File: PCB/bishi_pico.kicad_pcb (KiCad board)
At the start: 2 copper layers, 124 x 127.8 mm, 39 parts, among them SW1 SW_DIP_x01, SW2 SW_DIP_x01, SW3 SW_DIP_x01, SW4 SW_DIP_x01, U1 PiPico_No_SWD, U3 TMAG5273

Commit message: PCB v1.1 (ESD diodes added)
Parts:
- added TV1: ESD9B3.3ST5G, Diode_SMD:D_SOD-323_HandSoldering, F.Cu at (66.8, 90.0)
- added TV2: ESD9B3.3ST5G, Diode_SMD:D_SOD-323_HandSoldering, F.Cu at (73.1, 93.9)
- added TV3: ESD9B3.3ST5G, Diode_SMD:D_SOD-323_HandSoldering, F.Cu at (144.7, 95.9)
- added TV4: ESD9B3.3ST5G, Diode_SMD:D_SOD-323_HandSoldering, F.Cu at (158.5, 105.5)
- added TV5: ESD9B3.3ST5G, Diode_SMD:D_SOD-323_HandSoldering, F.Cu at (107.6, 68.8)
- added TV6: ESD9B3.3ST5G, Diode_SMD:D_SOD-323_HandSoldering, F.Cu at (110.6, 68.8)
- moved R1 3.00 mm to (113.4, 68.9)
- moved R2 2.91 mm to (104.6, 68.9)
Connections:
- net Net-(U1-USB1) renamed /USB_DN
- net Net-(U1-USB2) renamed /USB_DP
Routing:
- net /RX0: track 27.1 -> 36.2 mm
- net /RX1: track 108.6 -> 116.3 mm
- net /TX0: track 25.3 -> 32.3 mm
- net /TX1: track 107.0 -> 111.8 mm
- net /USB_DP: track 83.4 -> 86.3 mm
- net Net-(USB1-CC1): track 6.00 -> 8.41 mm
- net Net-(USB1-CC2): track 6.00 -> 8.37 mm
- net /USB_DN: track 81.1 -> 83.2 mm
Other:
- board text added: "v1.1"
- board text removed: "v1.0"
